File: BME680.kicad_pcb (KiCad board)
At the start: 2 copper layers, 25.4 x 17.8 mm, 20 parts, among them IC1 BME680, J1 HEADER-1X770MIL, Q2 BSS138, U2 AP2112K-3.3

Commit message: build(lib): use the kicad-common library
Parts:
- G***: footprint external_footprints:logo -> solar_cooker:solar_cooker_logo
Changed lines of the file:
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@@
 		)
 	)
-	(footprint "external_footprints:logo"
+	(footprint "solar_cooker:solar_cooker_logo"
 		(layer "F.Cu")
 		(at 157.5 105.44)
